File: noaa_filter/noaa_filter/noaa_filter.kicad_pcb (KiCad board)
At the start: 2 copper layers, 11 parts, among them J1 Conn_Coaxial, J2 Conn_Coaxial

Commit message: Working pcb
Parts:
- J1, J2: footprint Pin_Headers:Pin_Header_Straight_1x02_Pitch2.54mm -> lib:SMA-boardedge
- moved C5 37.0 mm to (97.5, 93.5), turned to 270 degrees
- moved J2 34.1 mm to (106.0, 91.4), turned to 180 degrees
- moved C7 31.5 mm to (100.3, 88.9)
- moved C6 31.4 mm to (93.5, 84.3)
- moved C3 29.8 mm to (89.4, 94.0)
- moved L1 29.4 mm to (84.8, 93.3)
- moved C1 28.4 mm to (81.9, 88.9)
- moved C4 28.2 mm to (91.4, 88.9)
- moved L2 27.9 mm to (97.5, 84.8)
- moved J1 26.2 mm to (76.2, 86.4), turned to 0 degrees
- moved C2 20.7 mm to (84.8, 84.8), turned to 90 degrees
Routing:
- net GND: vias 0 -> 10
- added copper zone on B.Cu, net GND
Other:
- board outline added: 36.1 x 21.3 mm
