File: noaa_filter/noaa_filter/noaa_filter.sch (KiCad schematic (older format))
At the start: 11 parts, among them J1 Conn_Coaxial, J2 Conn_Coaxial

Commit message: Working pcb
Parts:
- J1, J2: footprint Pin_Headers:Pin_Header_Straight_1x02_Pitch2.54mm -> lib:SMA-boardedge
Changed lines of the file:
@@
 EESchema Schematic File Version 4
+LIBS:noaa_filter-cache
 EELAYER 26 0
 EELAYER END
@@
 F 0 "J1" H 2700 3226 50  0000 L CNN
 F 1 "Conn_Coaxial" H 2700 3135 50  0000 L CNN
-F 2 "Pin_Headers:Pin_Header_Straight_1x02_Pitch2.54mm" H 2600 3250 50  0001 C CNN
+F 2 "lib:SMA-boardedge" H 2600 3250 50  0001 C CNN
 F 3 "" H 2600 3250 50  0001 C CNN
 	1    2600 3250
@@
 F 0 "J2" H 8900 3226 50  0000 L CNN
 F 1 "Conn_Coaxial" H 8900 3135 50  0000 L CNN
-F 2 "Pin_Headers:Pin_Header_Straight_1x02_Pitch2.54mm" H 8800 3250 50  0001 C CNN
+F 2 "lib:SMA-boardedge" H 8800 3250 50  0001 C CNN
 F 3 "" H 8800 3250 50  0001 C CNN
 	1    8800 3250
